Commit message: Updated for ASRS Robot URDF Integration

File: urdf/asrs_robot.xacro (robot description, xacro)
@@ -3,30 +3,23 @@
     <!-- Properties -->
     <xacro:property name="PI" value="3.14159265359" />
-    <!-- Material Definitions -->
-    <material name="blue">
-        <color rgba="0 0 1 1"/>
-    </material>
-    <material name="red">
-        <color rgba="1 0 0 1"/>
-    </material>
-    <material name="green">
-        <color rgba="0 1 0 1"/>
-    </material>
     <!-- Links -->
     <link name="world"/>
     <link name="base_link">
         <inertial>
-            <mass value="5.0"/>
-            <inertia ixx="0.1" ixy="0.0" ixz="0.0" iyy="0.1" iyz="0.0" izz="0.1"/>
+            <origin xyz="-0.00049298 0.038467 0.059588" rpy="0 0 0" />
+            <mass value="0.51487" />
+            <inertia ixx="0.00097956" ixy="8.6139E-07" ixz="-4.2275E-06" iyy="0.00063322" iyz="-6.2879E-06" izz="0.0014458" />
         </inertial>
         <visual>
             <geometry>
-                <cylinder length="0.2" radius="0.1"/>
+                <mesh filename="package://asrs_arm/meshes/link_1.STL"/>
             </geometry>
-            <material name="blue"/>
+            <material name=" ">
+                <color rgba="0.0 1.0 0.0 1.0"/>
+            </material>
         </visual>
         <collision>
             <geometry>
-                <cylinder length="0.2" radius="0.1"/>
+                <mesh filename="package://asrs_arm/meshes/link_1.STL"/>
             </geometry>
         </collision>
@@ -34,16 +27,19 @@
     <link name="shoulder_link">
         <inertial>
-            <mass value="3.0"/>
-            <inertia ixx="0.05" ixy="0.0" ixz="0.0" iyy="0.05" iyz="0.0" izz="0.05"/>
+            <origin xyz="3.3268E-05 0.038546 0.03493" rpy="0 0 0" />
+            <mass value="0.34286" />
+            <inertia ixx="0.0002982" ixy="-1.5865E-08" ixz="2.5289E-10" iyy="0.00012652" iyz="1.9537E-06" izz="0.0002767" />
         </inertial>
         <visual>
             <geometry>
-                <box size="0.3 0.05 0.05"/>
+                <mesh filename="package://asrs_arm/meshes/link_2.STL"/>
             </geometry>
-            <material name="red"/>
+            <material name=" ">
+                <color rgba="0.0 0.0 1.0 1.0"/>
+            </material>
         </visual>
         <collision>
             <geometry>
-                <box size="0.3 0.05 0.05"/>
+                <mesh filename="package://asrs_arm/meshes/link_2.STL"/>
             </geometry>
         </collision>
@@ -51,16 +47,19 @@
     <link name="elbow_link">
         <inertial>
-            <mass value="2.0"/>
-            <inertia ixx="0.02" ixy="0.0" ixz="0.0" iyy="0.02" iyz="0.0" izz="0.02"/>
+            <origin xyz="-0.00083473 -0.0061303 0.14093" rpy="0 0 0" />
+            <mass value="0.64592" />
+            <inertia ixx="0.00080618" ixy="-8.1896E-10" ixz="6.6639E-09" iyy="0.00073543" iyz="2.8682E-05" izz="0.00026191" />
         </inertial>
         <visual>
             <geometry>
-                <box size="0.2 0.05 0.05"/>
+                <mesh filename="package://asrs_arm/meshes/link_3.STL"/>
             </geometry>
-            <material name="green"/>
+            <material name=" ">
+                <color rgba="0.0 0.0 1.0 1.0"/>
+            </material>
         </visual>
         <collision>
             <geometry>
-                <box size="0.2 0.05 0.05"/>
+                <mesh filename="package://asrs_arm/meshes/link_3.STL"/>
             </geometry>
         </collision>
@@ -68,33 +67,19 @@
     <link name="wrist1_link">
         <inertial>
-            <mass value="1.0"/>
-            <inertia ixx="0.01" ixy="0.0" ixz="0.0" iyy="0.01" iyz="0.0" izz="0.01"/>
+            <origin xyz="0.00015398 -0.00014321 0.070552" rpy="0 0 0" />
+            <mass value="0.082446" />
+            <inertia ixx="7.1121E-05" ixy="-1.5741E-09" ixz="3.4653E-06" iyy="7.2808E-05" iyz="5.6573E-09" izz="1.4796E-05" />
         </inertial>
         <visual>
             <geometry>
-                <cylinder length="0.1" radius="0.025"/>
+                <mesh filename="package://asrs_arm/meshes/link_4.STL"/>
             </geometry>
-            <material name="blue"/>
+            <material name=" ">
+                <color rgba="0.0 0.0 1.0 1.0"/>
+            </material>
         </visual>
         <collision>
             <geometry>
-                <cylinder length="0.1" radius="0.025"/>
-            </geometry>
-        </collision>
-    </link>
-    <link name="tcp_link">
-        <inertial>
-            <mass value="0.5"/>
-            <inertia ixx="0.005" ixy="0.0" ixz="0.0" iyy="0.005" iyz="0.0" izz="0.005"/>
-        </inertial>
-        <visual>
-            <geometry>
-                <sphere radius="0.025"/>
-            </geometry>
-            <material name="green"/>
-        </visual>
-        <collision>
-            <geometry>
-                <sphere radius="0.025"/>
+                <mesh filename="package://asrs_arm/meshes/link_4.STL"/>
             </geometry>
         </collision>
@@ -104,5 +89,5 @@
         <parent link="world"/>
         <child link="base_link"/>
-        <origin xyz="0 0 0.1" rpy="0 0 0"/>
+        <origin xyz="0 0 0" rpy="0 0 0"/>
         <axis xyz="0 0 1"/>
         <limit lower="-${PI}" upper="${PI}" effort="50.0" velocity="1.0"/>
@@ -111,26 +96,21 @@
         <parent link="base_link"/>
         <child link="shoulder_link"/>
-        <origin xyz="0 0 0.14415" rpy="${PI/2} 0 0"/>
+        <origin xyz="0 0 0.0863" rpy="0 0 -0.013059"/>
         <axis xyz="0 0 1"/>
-        <limit lower="0" upper="${PI}" effort="30.0" velocity="1.0"/>
+        <limit lower="-${PI}" upper="${PI}" effort="30.0" velocity="1.0"/>
     </joint>
     <joint name="shoulder_to_elbow" type="revolute">
         <parent link="shoulder_link"/>
         <child link="elbow_link"/>
-        <origin xyz="0.24381 0 0" rpy="0 0 0"/>
-        <axis xyz="0 0 1"/>
-        <limit lower="-${3*PI/4}" upper="0" effort="30.0" velocity="1.0"/>
+        <origin xyz="0 0 0.07095" rpy="0 0 0"/>
+        <axis xyz="-1.0 0.0 0"/>
+        <limit lower="-${PI/4}" upper="${PI/4}" effort="30.0" velocity="1.0"/>
     </joint>
     <joint name="elbow_to_wrist1" type="revolute">
         <parent link="elbow_link"/>
         <child link="wrist1_link"/>
-        <origin xyz="0.12475 0 0" rpy="0 0 0"/>
-        <axis xyz="0 0 1"/>
-        <limit lower="-${PI/2}" upper="${PI/2}" effort="20.0" velocity="1.0"/>
-    </joint>
-    <joint name="wrist1_to_tcp" type="fixed">
-        <parent link="wrist1_link"/>
-        <child link="tcp_link"/>
-        <origin xyz="0.08475 0 0" rpy="-${PI/2} 0 0"/>
+        <origin xyz="0.0083376 -0.030916 0.24181" rpy="0.96329 0.012835 0.018459"/>
+        <axis xyz="1.0 0.0 0"/>
+        <limit lower="-${PI/4}" upper="${PI/4}" effort="20.0" velocity="1.0"/>
     </joint>
 </robot>

Commit message: updates in urdf files and paths

File: urdf/asrs_robot.xacro (robot description, xacro)
@@ -13,5 +13,5 @@
         <visual>
             <geometry>
-                <mesh filename="package://asrs_arm/meshes/link_1.STL"/>
+                <mesh filename="package://my_robot_arm/meshes/link_1.STL"/>
             </geometry>
             <material name=" ">
@@ -21,5 +21,5 @@
         <collision>
             <geometry>
-                <mesh filename="package://asrs_arm/meshes/link_1.STL"/>
+                <mesh filename="package://my_robot_arm/meshes/link_1.STL"/>
             </geometry>
         </collision>
@@ -33,5 +33,5 @@
         <visual>
             <geometry>
-                <mesh filename="package://asrs_arm/meshes/link_2.STL"/>
+                <mesh filename="package://my_robot_arm/meshes/link_2.STL"/>
             </geometry>
             <material name=" ">
@@ -41,5 +41,5 @@
         <collision>
             <geometry>
-                <mesh filename="package://asrs_arm/meshes/link_2.STL"/>
+                <mesh filename="package://my_robot_arm/meshes/link_2.STL"/>
             </geometry>
         </collision>
@@ -53,5 +53,5 @@
         <visual>
             <geometry>
-                <mesh filename="package://asrs_arm/meshes/link_3.STL"/>
+                <mesh filename="package://my_robot_arm/meshes/link_3.STL"/>
             </geometry>
             <material name=" ">
@@ -61,5 +61,5 @@
         <collision>
             <geometry>
-                <mesh filename="package://asrs_arm/meshes/link_3.STL"/>
+                <mesh filename="package://my_robot_arm/meshes/link_3.STL"/>
             </geometry>
         </collision>
@@ -73,5 +73,5 @@
         <visual>
             <geometry>
-                <mesh filename="package://asrs_arm/meshes/link_4.STL"/>
+                <mesh filename="package://my_robot_arm/meshes/link_4.STL"/>
             </geometry>
             <material name=" ">
@@ -81,5 +81,5 @@
         <collision>
             <geometry>
-                <mesh filename="package://asrs_arm/meshes/link_4.STL"/>
+                <mesh filename="package://my_robot_arm/meshes/link_4.STL"/>
             </geometry>
         </collision>
