Commit message: Added new README with assets, updated launch and urdf files
Added new README.md and updated URDF and launch files

File: urdf/asrs_robots.xacro (robot description, xacro)
@@ -86,10 +86,10 @@
   </link>
   <!-- ARM JOINTS -->
-  <joint name="world_to_baselink" type="revolute">
+  <joint name="world_to_baselink" type="fixed">
     <parent link="world"/>
     <child link="base_link"/>
     <origin xyz="0 0 0" rpy="0 0 0"/>
     <axis xyz="0 0 1"/>
-    <limit lower="-${PI}" upper="${PI}" effort="50.0" velocity="1.0"/>
+    <!--<limit lower="-${PI}" upper="${PI}" effort="50.0" velocity="1.0"/> -->
   </joint>
   <joint name="base_to_shoulder" type="revolute">
@@ -117,8 +117,10 @@
   <!-- 1. Attach gripper fixture to the wrist -->
   <link name="gripper_fixture" />
-  <joint name="wrist1_to_gripper_fixture" type="fixed">
+  <joint name="wrist1_to_gripper_fixture" type="revolute">
     <parent link="wrist1_link"/>
     <child link="gripper_fixture"/>
     <origin xyz="-0.02866 0.0 0.12448" rpy="0 0 0"/>
+    <axis xyz="1.0 0.0 0"/>
+    <limit lower="-${PI/4}" upper="${PI/4}" effort="20.0" velocity="1.0"/>
   </joint>
   <!-- 2. Gripper Base (equivalent to "base" in the reference, renamed to avoid confusion) -->
@@ -177,9 +179,14 @@
   </link>
   <!-- Fixed joint connecting gripper_base to gripper_driver -->
-  <joint name="gripper_base_to_driver" type="fixed">
+  <joint name="gripper_base_to_driver" type="revolute">
     <parent link="gripper_base"/>
     <child link="gripper_driver"/>
     <origin xyz="-0.018617 0.020144 -0.00018182" rpy="0 0 0"/>
     <axis xyz="0 0 -1"/>
+    <limit
+      lower="10.0"
+      upper="${PI/4}"
+      effort="0"
+      velocity="0.5" />
   </joint>
   <!-- 4. Left Finger -->
@@ -208,5 +215,5 @@
   </link>
   <!-- Joint connecting gripper_driver to left_finger -->
-  <joint name="driver_to_left_finger" type="fixed">
+  <joint name="driver_to_left_finger" type="continuous">
     <parent link="gripper_driver"/>
     <child link="left_finger"/>
@@ -240,5 +247,5 @@
   </link>
   <!-- Fixed joint connecting gripper_base to gripper_driven -->
-  <joint name="gripper_base_to_driven" type="fixed">
+  <joint name="gripper_base_to_driven" type="continuous">
     <parent link="gripper_base"/>
     <child link="gripper_driven"/>
@@ -272,5 +279,5 @@
   </link>
   <!-- Joint connecting gripper_driven to right_finger -->
-  <joint name="driven_to_right_finger" type="fixed">
+  <joint name="driven_to_right_finger" type="continuous">
     <parent link="gripper_driven"/>
     <child link="right_finger"/>
@@ -304,5 +311,5 @@
   </link>
   <!-- Joint connecting gripper_base to left_knuckle -->
-  <joint name="gripper_base_to_left_knuckle" type="fixed">
+  <joint name="gripper_base_to_left_knuckle" type="continuous">
     <parent link="gripper_base"/>
     <child link="left_knuckle"/>
@@ -335,5 +342,5 @@
   </link>
   <!-- Joint connecting gripper_base to right_knuckle -->
-  <joint name="gripper_base_to_right_knuckle" type="fixed">
+  <joint name="gripper_base_to_right_knuckle" type="continuous">
     <parent link="gripper_base"/>
     <child link="right_knuckle"/>
@@ -342,3 +349,28 @@
     <mimic joint="gripper_base_to_driver" multiplier="1" offset="0"/>
   </joint>
+  <ros2_control name="asrs_robot_control" type="system">
+  <hardware>
+    <plugin>ros2_control_demo_hardware/GenericSystem</plugin>
+  </hardware>
+  <joint name="base_to_shoulder">
+    <command_interface name="position"/>
+    <state_interface name="position"/>
+    <state_interface name="velocity"/>
+  </joint>
+  <joint name="shoulder_to_elbow">
+    <command_interface name="position"/>
+    <state_interface name="position"/>
+    <state_interface name="velocity"/>
+  </joint>
+  <joint name="elbow_to_wrist1">
+    <command_interface name="position"/>
+    <state_interface name="position"/>
+    <state_interface name="velocity"/>
+  </joint>
+  <joint name="wrist1_to_gripper_fixture">
+    <command_interface name="position"/>
+    <state_interface name="position"/>
+    <state_interface name="velocity"/>
+  </joint>
+ </ros2_control>
 </robot>
